File: PCBs/DNMS-T4.0+NodeMCU/DNMS-T4.0+NodeMCU-V1.4/DNMS.kicad_pcb (KiCad board)
At the start: 2 copper layers, 137.2 x 33.6 mm, 17 parts, among them J1 Conn_02x03_Odd_Even, J2 Conn_01x02, J3 Conn_01x04, J4 Conn_01x05, U1 NodeMCU V2, U2 NodeMCU V3, U3 Teensy4.0

Commit message: Änderungen im Bestückungsdruck/change of silkscreen
Other:
- board text added: "+3.3V"
- board text added: "I²C"
- board text added: "SCL"
- board text added: "SDA"
Changed lines of the file:
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@@
   (general
     (thickness 1.6)
-    (drawings 20)
+    (drawings 25)
     (tracks 265)
     (zones 0)
@@
     (descr "Through hole straight pin header, 1x04, 2.54mm pitch, single row")
     (tags "Through hole pin header THT 1x04 2.54mm single row")
-    (fp_text reference J3 (at 0.00762 -10.60958 180) (layer B.SilkS)
+    (fp_text reference J3 (at 0.86244 -10.49858 180) (layer B.SilkS)
       (effects (font (size 1 1) (thickness 0.15)) (justify mirror))
     )
@@
     )
   )
+  (gr_text I²C (at 136.53262 65.74282) (layer B.SilkS)
+    (effects (font (size 1 1) (thickness 0.15)) (justify mirror))
+  )
+  (gr_text SDA (at 133.26364 63.08344 90) (layer B.SilkS)
+    (effects (font (size 1 1) (thickness 0.15)) (justify mirror))
+  )
+  (gr_text SCL (at 130.86842 63.12408 90) (layer B.SilkS)
+    (effects (font (size 1 1) (thickness 0.15)) (justify mirror))
+  )
+  (gr_text GND (at 128.41224 63.1444 90) (layer B.SilkS)
+    (effects (font (size 1 1) (thickness 0.15)) (justify mirror))
+  )
+  (gr_text +3.3V (at 125.9967 62.31128 90) (layer B.SilkS)
+    (effects (font (size 1 1) (thickness 0.15)) (justify mirror))
+  )
   (gr_text SPS30 (at 116.34724 60.1726) (layer B.SilkS)
