File: PCBs/DNMS-T4.0/DNMS-T4.0-V1.7/DNMS.kicad_pcb (KiCad board)
At the start: 2 copper layers, 131.1 x 19.2 mm, 21 parts, among them J1 Conn_01x02, J2 Conn_02x03_Odd_Even, J3 Conn_01x04, J4 Conn_01x01, J5 RJ12, J6 RJ12, J7 SM06B-SRSS-TB(LF)(SN), J8 SM06B-SRSS-TB(LF)(SN), U1 Teensy4.0, U2 P82B715PN,112, U3 P82B715DR

Commit message: new firmware
Parts:
- removed G***: LOGO, logos eigene:logo luftdaten.info
- removed REF1 (x4): MountingHole_2.7mm_M2.5, MountingHole:MountingHole_2.7mm_M2.5
- J5: footprint Connector_RJ:RJ12_Amphenol_54601 -> 54601906WPLF:54601906WPLF
- J6: footprint Connector_RJ:RJ12_Pulse_E5566Q0LK22L -> E5566-Q0LK22-L:E5566Q0LK22L
- U2: footprint P82B715PN_112:DIP254P762X420-8 -> P82B715:DIP254P762X420-8
