File: PCBs/DNMS-T4.0/DNMS-T4.0-V1.7/DNMS.kicad_sch (KiCad schematic)
At the start: 16 parts, among them J1 Conn_01x02, J2 Conn_02x03_Odd_Even, J3 Conn_01x04, J4 Conn_01x01, J5 RJ12, J6 RJ12, J7 SM06B-SRSS-TB(LF)(SN), J8 SM06B-SRSS-TB(LF)(SN), U1 Teensy4.0, U2 P82B715PN,112, U3 P82B715DR

Commit message: new firmware
Parts:
- U2: footprint P82B715PN_112:DIP254P762X420-8 -> P82B715:DIP254P762X420-8
Connections:
- no-connect marks 24 -> 23
