File: PCBs/IM72D128 microphone PCB/IM72D128-PCB-V1.0/IM72D128-PCB.kicad_pcb (KiCad board)
At the start: 2 copper layers, 11.3 x 11.3 mm, 8 parts

Commit message: new firmware
Parts:
- SP2: value CLK -> CLOCK
- SP3: value SEL -> SELECT
