File: PCBs/IM72D128 microphone PCB/IM72D128-PCB-V1.0/IM72D128-PCB.kicad_sch (KiCad schematic)
At the start: 8 parts

Commit message: new firmware
Parts:
- SP2: value CLK -> CLOCK
- SP3: value SEL -> SELECT
