File: PCBs/IM72D128 microphone PCB/IM72D128-Tube-PCB-V1.0/IM72D128-Tube-PCB.kicad_pcb (KiCad board)
At the start: 2 copper layers, 130 x 11 mm, 23 parts, among them J1 Conn_02x03_Odd_Even, U1 LP5907MFX-3.3, U2 ADAU7002ACBZ-R7, U3 SN74LV1T34DBVR, U4 SN74LV1T34DBVR, U5 SN74LV1T34DBVR

Commit message: new firmware
Parts:
- SP3: value SEL -> SELECT
